Commit message: Add files via upload

File: ros2_ws/src/cobraflex/urdf/rplidar_a2.urdf.xacro (robot description, xacro)
@@ -1,17 +1,68 @@
 <?xml version="1.0"?>
 <robot xmlns:xacro="http://www.ros.org/wiki/xacro">
-  <xacro:macro name="rplidar_a2" params="parent xyz rpy">
     <link name="lidar_link">
       <visual>
+        <origin xyz="0 0 0" rpy="0 0 0"/>
         <geometry>
-          <cylinder radius="0.04" length="0.06"/>
+          <cylinder radius="0.0375" length="0.05"/>
         </geometry>
+        <material name="green">
+            <color rgba="0.003 0.639 0.223 1.0"/>
+        </material>
       </visual>
+      <collision>
+        <origin xyz="0 0 0" rpy="0 0 0"/>
+        <geometry>
+          <cylinder radius="0.0375" length="0.05"/>
+        </geometry>
+      </collision>
+      <inertial>
+        <origin xyz="0 0 0" rpy="0 0 0"/>
+        <mass value="0.1"/>
+        <inertia ixx="${(2/5) * 0.1 * (0.0375 * 0.0375)}" ixy="0" ixz="0"
+                 iyy="${(2/5) * 0.1 * (0.0375 * 0.0375)}" iyz="0"
+                 izz="${(2/5) * 0.1 * (0.0375 * 0.0375)}" />
+      </inertial>
     </link>
-    <joint name="base_to_lidar" type="fixed">
-      <parent link="${parent}"/>
+    <joint name="lidar_to_base_link" type="fixed">
+      <parent link="base_link"/>
       <child link="lidar_link"/>
-      <origin xyz="${xyz}" rpy="${rpy}"/>
+      <origin xyz="0 0 0.16" rpy="0 0 0"/>
     </joint>
-  </xacro:macro>
+    <gazebo reference="lidar_link">
+      <sensor name="gpu_lidar" type="gpu_lidar">
+        <topic>scan</topic>
+        <gz_frame_id>lidar_link</gz_frame_id>
+        <update_rate>10</update_rate>
+        <always_on>true</always_on>
+        <visualize>true</visualize>
+        <ray>
+          <scan>
+            <horizontal>
+              <samples>720</samples>
+              <resolution>0.01</resolution>
+              <min_angle>-3.1416</min_angle>
+              <max_angle>3.1416</max_angle>
+            </horizontal>
+            <vertical>
+              <samples>1</samples>
+              <resolution>1</resolution>
+              <min_angle>0.0</min_angle>
+              <max_angle>0.0</max_angle>
+            </vertical>
+          </scan>
+          <range>
+            <min>0.2</min>
+            <max>20.0</max>
+            <resolution>0.01</resolution>
+          </range>
+        </ray>
+      </sensor>
+    </gazebo>
+    <link name="my_robot/base_footprint/gpu_lidar"/>
+    <joint name="lidar_joint" type="fixed">
+        <parent link="lidar_link" />
+        <child link="my_robot/base_footprint/gpu_lidar" />
+        <origin xyz="0 0 0" rpy="0 0 0" />
+    </joint>
 </robot>
