Commit message: Guide check workflow

File: src/cobraflex/urdf/my_robot_gazebo_mesh.urdf (robot description, URDF)
Before this commit: robot cobraflex_robot, 7 links, 7 joints
Joints:
- joint camera_joint_lane: origin xyz=${body_length/2 + 0.02} 0 -0.03 rpy=0 0 0 -> xyz=${body_length/2 + 0.01} 0 -0.03 rpy=0 0.30 0

Commit message: Cobraflex V4 update

File: src/cobraflex/urdf/my_robot_gazebo_mesh.urdf (robot description, URDF)
Before this commit: robot cobraflex_robot, 7 links, 7 joints
Links:
- link lidar_link: geometry collision cylinder length=0.04 radius=0.0375; visual mesh filename=file://$(find cobraflex)/meshes/rplidar-a2m4-r1_hull.stl scale=0.001 0.001 0.001

File: src/cobraflex/urdf/my_robot_mesh.urdf (robot description, URDF)
Before this commit: robot cobraflex_robot, 10 links, 9 joints
Links:
- link lidar_link: geometry collision cylinder length=0.04 radius=0.0375; visual mesh filename=file://$(find cobraflex)/meshes/rplidar-a2m4-r1_hull.stl scale=0.001 0.001 0.001
