Commit message: Refactor navigation launch and configuration files; update URDF mass properties and add new maps and worlds documentation
- Updated `navigation.launch.py` to use package-relative paths for map and parameters files.
- Added `nav2_params.yaml` for customized navigation parameters specific to the CobraFlex platform.
- Created `README.md` in `maps/` directory to guide users on saving and using occupancy grids.
- Added `README.md` in `worlds/` directory detailing available SDF worlds for Gazebo and instructions for adding new worlds.
- Adjusted mass properties in URDF files to reflect accurate weights for the chassis and body components.
- Updated maintainer information and license type in `package.xml` and `setup.py` files across multiple packages.
- Added missing files and directories to `setup.py` to ensure proper installation of URDF and mesh assets.

File: src/cobraflex/urdf/cobraflex_isaac.urdf (robot description, URDF)
Before this commit: robot cobraflex_robot, 17 links, 16 joints
Links:
- link base_link: mass 5.0 -> 2.20
- link body_link: mass 1.0 -> 0.71

Commit message: Repo Update

File: src/cobraflex/urdf/cobraflex_isaac.urdf (robot description, URDF)
Before this commit: robot cobraflex_robot, 17 links, 16 joints
Links:
- link base_link: mass 2.20 -> 2.0172
- link body_link: mass 0.71 -> 0.8928

Commit message: Cobraflex V4

File: src/cobraflex/urdf/cobraflex_isaac.urdf (robot description, URDF)
Before this commit: robot cobraflex_robot, 17 links, 16 joints
Links:
- link body_link: geometry collision box size=0.102 0.1299 0.057; collision box size=0.18 0.0995 0.0255
Joints:
- joint imu_joint: origin xyz=0.0665 0 0.02 rpy=0 0 0 -> xyz=0.0882 0 0.02505 rpy=0 0.2618 0
- joint lidar_joint: origin xyz=0 0 0.09 rpy=0 0 0 -> xyz=0.035 0 0.0458 rpy=0 0 3.141592653589793
- joint zedm_left_camera_joint: origin xyz=0.02 0.0245 0 rpy=0 0 0 -> xyz=0.02 0.02375 0 rpy=0 0 0
- joint zedm_mount_joint: origin xyz=0.0665 0 0.006750000000000001 rpy=0 0 0 -> xyz=0.0848 0 0.01225 rpy=0 0.2618 0
- joint zedm_right_camera_joint: origin xyz=0.02 -0.0385 0 rpy=0 0 0 -> xyz=0.02 -0.03925 0 rpy=0 0 0

File: src/cobraflex/urdf/my_robot_basic.urdf (robot description, URDF)
Before this commit: robot cobraflex_robot, 23 links, 23 joints
Links:
- removed link viz_lidar_standoffs
- removed link viz_mast_plate
- link body_link: geometry collision box size=0.102 0.1299 0.057; collision box size=0.18 0.0995 0.0255
- link viz_deck_hardware: geometry visual box size=0.082 0.082 0.010
- link viz_jetson: geometry visual box size=0.099 0.090 0.025
Joints:
- removed joint viz_lidar_standoffs_joint
- removed joint viz_mast_plate_joint
- joint body_joint: origin xyz=0 0 ${body_height/2 + chassis_height/2} -> xyz=0 0 ${body_link_z - wheel_radius}
- joint imu_joint: origin xyz=${body_length/2 - 0.04} 0 0.02 rpy=0 0 0 -> xyz=${zed_center_x} 0 ${zed_center_z - body_link_z} rpy=0 ${zed_pitch} 0
- joint lidar_joint: origin xyz=0 0 ${body_height/2 + 0.04} rpy=0 0 ${pi} -> xyz=${lidar_scan_x} 0 ${lidar_scan_z - body_link_z} rpy=0 0 ${pi}
- joint zed_mount_joint: origin xyz=0.11 0 0.02 rpy=0 0 0 -> xyz=${zed_mount_x} 0 ${zed_mount_z - body_link_z} rpy=0 ${zed_pitch} 0

File: src/cobraflex/urdf/my_robot_gazebo.urdf (robot description, URDF)
Before this commit: robot cobraflex_robot, 7 links, 7 joints
Links:
- link body_link: geometry collision box size=0.102 0.1299 0.057; collision box size=0.18 0.0995 0.0255
Joints:
- joint body_joint: origin xyz=0 0 ${body_height/2 + chassis_height/2} -> xyz=0 0 ${body_link_z - wheel_radius}
- joint imu_joint: origin xyz=${body_length/2 - 0.04} 0 0.02 rpy=0 0 0 -> xyz=${zed_center_x} 0 ${zed_center_z - body_link_z} rpy=0 ${zed_pitch} 0
- joint lidar_joint: origin xyz=0 0 ${body_height/2 + 0.04} rpy=0 0 ${pi} -> xyz=${lidar_scan_x} 0 ${lidar_scan_z - body_link_z} rpy=0 0 ${pi}
- joint zedm_mount_joint: origin xyz=${body_length/2 - 0.0475} 0 ${0.02 - 0.0265/2} rpy=0 0 0 -> xyz=${zed_mount_x} 0 ${zed_mount_z - body_link_z} rpy=0 ${zed_pitch} 0

File: src/cobraflex/urdf/my_robot_gazebo_mesh.urdf (robot description, URDF)
Before this commit: robot cobraflex_robot, 7 links, 7 joints
Links:
- link body_link: geometry collision box size=0.102 0.1299 0.057; collision box size=0.18 0.0995 0.0255
Joints:
- joint body_joint: origin xyz=0 0 ${body_height/2 + chassis_height/2 - 0.01} -> xyz=0 0 ${body_link_z - wheel_radius}
- joint imu_joint: origin xyz=${body_length/2 - 0.0475} 0 0.02 rpy=0 0 0 -> xyz=${zed_center_x} 0 ${zed_center_z - body_link_z} rpy=0 ${zed_pitch} 0
- joint lidar_joint: origin xyz=0 0 ${body_height/2 + 0.04} rpy=0 0 0 -> xyz=${lidar_scan_x} 0 ${lidar_scan_z - body_link_z} rpy=0 0 ${pi}
- joint zedm_mount_joint: origin xyz=${body_length/2 - 0.0475} 0 ${0.02 - 0.0265/2} rpy=0 0 0 -> xyz=${zed_mount_x} 0 ${zed_mount_z - body_link_z} rpy=0 ${zed_pitch} 0

File: src/cobraflex/urdf/my_robot_mesh.urdf (robot description, URDF)
Before this commit: robot cobraflex_robot, 10 links, 9 joints
Links:
- link body_link: geometry collision box size=0.102 0.1299 0.057; collision box size=0.18 0.0995 0.0255
Joints:
- joint body_joint: origin xyz=0 0 ${body_height/2 + chassis_height/2 - 0.01} -> xyz=0 0 ${body_link_z - wheel_radius}
- joint camera_joint: origin xyz=${body_length/2 - 0.0475} 0 0.02 rpy=0 0 0 -> xyz=${zed_center_x} 0 ${zed_center_z - body_link_z} rpy=0 ${zed_pitch} 0
- joint imu_joint: origin xyz=${body_length/2 - 0.0475} 0 0.02 rpy=0 0 0 -> xyz=${zed_center_x} 0 ${zed_center_z - body_link_z} rpy=0 ${zed_pitch} 0
- joint lidar_joint: origin xyz=0 0 ${body_height/2 + 0.04} rpy=0 0 0 -> xyz=${lidar_scan_x} 0 ${lidar_scan_z - body_link_z} rpy=0 0 ${pi}

File: src/cobraflex/urdf/zed_macro.urdf.xacro (robot description, xacro)
@@ -212,8 +212,10 @@
         </xacro:if>
       </link>
+      <!-- Lens positions of the ZED Mini: 0.02 m ahead of the camera centre (middle of the
+           housing) and 7.75 mm to its right (camera CAD model and Stereolabs zedm.stl). -->
       <joint name="${name}_left_camera_joint" type="fixed">
         <parent link="${name}_camera_center"/>
         <child link="${name}_left_camera_frame"/>
-        <origin xyz="${optical_offset_x + 0.02} ${baseline/2 - 0.007} 0" rpy="0 0 0" />
+        <origin xyz="${optical_offset_x + 0.02} ${baseline/2 - 0.00775} 0" rpy="0 0 0" />
       </joint>
       <link name="${name}_left_camera_frame_optical"/>
@@ -246,5 +248,5 @@
         <parent link="${name}_camera_center"/>
         <child link="${name}_right_camera_frame"/>
-        <origin xyz="${optical_offset_x + 0.02} -${baseline/2 + 0.007} 0" rpy="0 0 0" />
+        <origin xyz="${optical_offset_x + 0.02} -${baseline/2 + 0.00775} 0" rpy="0 0 0" />
       </joint>
       <link name="${name}_right_camera_frame_optical"/>

Commit message: Cobraflex V4 update

File: src/cobraflex/urdf/cobraflex_isaac.urdf (robot description, URDF)
Before this commit: robot cobraflex_robot, 17 links, 16 joints
Links:
- link base_link: geometry collision box size=0.228 0.13 0.074; visual mesh filename=../meshes/cobraflex_chassis.stl scale=0.001 0.001 0.001

File: src/cobraflex/urdf/my_robot_basic.urdf (robot description, URDF)
Before this commit: robot cobraflex_robot, 21 links, 21 joints
Links:
- removed link viz_bumpers
- removed link viz_chassis_rails
- removed link viz_deck_hardware
- removed link viz_drivetrain
- removed link viz_jetson
- removed link viz_lane_cam_lens
- removed link viz_lidar_aperture
- removed link viz_lidar_head
- removed link viz_lipo
- removed link viz_motor
- removed link viz_servo
- removed link viz_skirts
- link base_link: geometry collision box size=${chassis_length} ${chassis_width} ${chassis_box_height}; visual box size=${chassis_length} ${chassis_width} ${chassis_box_height}
- link camera_link_lane: geometry collision box size=0.005 0.02 0.02; visual box size=0.004 0.025 0.024
- link lidar_link: geometry collision cylinder length=0.04 radius=0.0375; visual box size=0.012 0.024 0.013
Joints:
- removed joint viz_bumpers_joint
- removed joint viz_chassis_rails_joint
- removed joint viz_deck_hardware_joint
- removed joint viz_drivetrain_joint
- removed joint viz_jetson_joint
- removed joint viz_lane_cam_lens_joint
- removed joint viz_lidar_aperture_joint
- removed joint viz_lidar_head_joint
- removed joint viz_lipo_joint
- removed joint viz_motor_joint
- removed joint viz_servo_joint
- removed joint viz_skirts_joint

File: src/cobraflex/urdf/my_robot_gazebo.urdf (robot description, URDF)
Before this commit: robot cobraflex_robot, 7 links, 7 joints
Links:
- link base_link: geometry collision box size=${chassis_length} ${chassis_width} ${chassis_box_height}; visual box size=${chassis_length} ${chassis_width} ${chassis_box_height}

File: src/cobraflex/urdf/my_robot_gazebo_mesh.urdf (robot description, URDF)
Before this commit: robot cobraflex_robot, 7 links, 7 joints
Links:
- link base_link: geometry collision box size=${chassis_length} ${chassis_width} ${chassis_box_height}; visual mesh filename=file://$(find cobraflex)/meshes/cobraflex_chassis.stl scale=0.001 0.001 0.001

File: src/cobraflex/urdf/my_robot_mesh.urdf (robot description, URDF)
Before this commit: robot cobraflex_robot, 10 links, 9 joints
Links:
- link base_link: geometry collision box size=${chassis_length} ${chassis_width} ${chassis_box_height}; visual mesh filename=file://$(find cobraflex)/meshes/cobraflex_chassis.stl scale=0.001 0.001 0.001

Commit message: Cobraflex V4 update

File: src/cobraflex/urdf/cobraflex_isaac.urdf (robot description, URDF)
Before this commit: robot cobraflex_robot, 17 links, 16 joints
Joints:
- joint camera_joint_lane: origin xyz=0.124 0 -0.03 rpy=0 0.30 0 -> xyz=0.13 0 -0.03 rpy=0 0.30 0

File: src/cobraflex/urdf/my_robot_basic.urdf (robot description, URDF)
Before this commit: robot cobraflex_robot, 9 links, 9 joints
Joints:
- joint camera_joint_lane: origin xyz=${body_length/2 + 0.01} 0 -0.03 rpy=0 0.3 0 -> xyz=0.13 0 -0.03 rpy=0 0.3 0

File: src/cobraflex/urdf/my_robot_gazebo.urdf (robot description, URDF)
Before this commit: robot cobraflex_robot, 7 links, 7 joints
Joints:
- joint camera_joint_lane: origin xyz=${body_length/2 + 0.01} 0 -0.03 rpy=0 0.30 0 -> xyz=0.13 0 -0.03 rpy=0 0.30 0

File: src/cobraflex/urdf/my_robot_gazebo_mesh.urdf (robot description, URDF)
Before this commit: robot cobraflex_robot, 7 links, 7 joints
Joints:
- joint camera_joint_lane: origin xyz=${body_length/2 + 0.01} 0 -0.03 rpy=0 0.30 0 -> xyz=0.13 0 -0.03 rpy=0 0.30 0

File: src/cobraflex/urdf/my_robot_mesh.urdf (robot description, URDF)
Before this commit: robot cobraflex_robot, 10 links, 9 joints
Joints:
- joint camera_joint_lane: origin xyz=${body_length/2 + 0.01} 0 -0.03 rpy=0 0.30 0 -> xyz=0.13 0 -0.03 rpy=0 0.30 0
