Commit message: Repo Update

File: src/cobraflex/urdf/my_robot_basic.urdf (robot description, URDF)
Before this commit: robot cobraflex_robot, 7 links, 7 joints
Links:
- added link camera_link_lane; collision box size=0.005 0.02 0.02; visual box size=0.004 0.025 0.024
- added link camera_link_optical_lane
- added link viz_bumpers; visual box size=0.020 0.116 0.020; visual box size=0.022 0.124 0.020
- added link viz_chassis_rails; visual box size=0.170 0.020 0.034; visual box size=0.170 0.020 0.034
- added link viz_deck_hardware; visual box size=0.082 0.082 0.014; visual cylinder length=0.086 radius=0.0035
- added link viz_drivetrain; visual cylinder length=0.049 radius=0.006; visual cylinder length=0.049 radius=0.006
- added link viz_jetson; visual box size=0.105 0.092 0.043
- added link viz_lane_cam_lens; visual cylinder length=0.001 radius=0.0034; visual cylinder length=0.009 radius=0.0055
- added link viz_lidar_aperture; visual box size=0.012 0.024 0.013
- added link viz_lidar_head; visual cylinder length=0.018 radius=0.0350
- added link viz_lidar_standoffs; visual cylinder length=0.020 radius=0.003; visual cylinder length=0.020 radius=0.003
- added link viz_lipo; visual box size=0.078 0.046 0.028
- added link viz_mast_plate; visual box size=0.014 0.100 0.008
- added link viz_motor; visual cylinder length=0.048 radius=0.0165
- added link viz_servo; visual box size=0.040 0.021 0.037
- added link viz_skirts; visual box size=0.190 0.008 0.048; visual box size=0.190 0.008 0.048
- link base_link: geometry collision box size=${chassis_length} ${chassis_width} ${chassis_height}; visual box size=${chassis_length} 0.112 0.010
- link body_link: geometry collision box size=${body_length} ${body_width} ${body_height}; visual box size=${body_length} 0.176 0.008
- link camera_link: geometry collision box size=0.01 0.1 0.02
- link lidar_link: geometry collision cylinder length=0.04 radius=0.0375; visual cylinder length=0.012 radius=0.0375
Joints:
- removed joint footprint_joint
- added joint camera_joint_lane: type fixed, parent body_link, child camera_link_lane, origin xyz=${body_length/2 + 0.01} 0 -0.03 rpy=0 0.3 0
- added joint camera_optical_joint_lane: type fixed, parent camera_link_lane, child camera_link_optical_lane, origin xyz=0 0 0 rpy=${-pi/2} 0 ${-pi/2}
- added joint viz_bumpers_joint: type fixed, parent base_link, child viz_bumpers, origin xyz=0 0 0 rpy=0 0 0
- added joint viz_chassis_rails_joint: type fixed, parent base_link, child viz_chassis_rails, origin xyz=0 0 0 rpy=0 0 0
- added joint viz_deck_hardware_joint: type fixed, parent body_link, child viz_deck_hardware, origin xyz=0 0 0 rpy=0 0 0
- added joint viz_drivetrain_joint: type fixed, parent base_link, child viz_drivetrain, origin xyz=0 0 0 rpy=0 0 0
- added joint viz_jetson_joint: type fixed, parent body_link, child viz_jetson, origin xyz=0 0 0 rpy=0 0 0
- added joint viz_lane_cam_lens_joint: type fixed, parent camera_link_lane, child viz_lane_cam_lens, origin xyz=0 0 0 rpy=0 0 0
- added joint viz_lidar_aperture_joint: type fixed, parent lidar_link, child viz_lidar_aperture, origin xyz=0 0 0 rpy=0 0 0
- added joint viz_lidar_head_joint: type fixed, parent lidar_link, child viz_lidar_head, origin xyz=0 0 0 rpy=0 0 0
- added joint viz_lidar_standoffs_joint: type fixed, parent lidar_link, child viz_lidar_standoffs, origin xyz=0 0 0 rpy=0 0 0
- added joint viz_lipo_joint: type fixed, parent body_link, child viz_lipo, origin xyz=0 0 0 rpy=0 0 0
- added joint viz_mast_plate_joint: type fixed, parent body_link, child viz_mast_plate, origin xyz=0 0 0 rpy=0 0 0
- added joint viz_motor_joint: type fixed, parent base_link, child viz_motor, origin xyz=0 0 0 rpy=0 0 0
- added joint viz_servo_joint: type fixed, parent base_link, child viz_servo, origin xyz=0 0 0 rpy=0 0 0
- added joint viz_skirts_joint: type fixed, parent body_link, child viz_skirts, origin xyz=0 0 0 rpy=0 0 0
- added joint zed_mount_joint: type fixed, parent body_link, child zed_camera_link, origin xyz=0.11 0 0.02 rpy=0 0 0

File: src/cobraflex/urdf/my_robot_gazebo.urdf (robot description, URDF)
Before this commit: robot cobraflex_robot, 7 links, 6 joints
Links:
- removed link camera_link
- removed link camera_link_optical
- added link camera_link_lane; collision cylinder length=0.002 radius=0.005; visual cylinder length=0.002 radius=0.005
- added link camera_link_optical_lane
Joints:
- removed joint camera_joint
- removed joint camera_optical_joint
- added joint camera_joint_lane: type fixed, parent body_link, child camera_link_lane, origin xyz=${body_length/2 + 0.01} 0 -0.03 rpy=0 0.30 0
- added joint camera_optical_joint_lane: type fixed, parent camera_link_lane, child camera_link_optical_lane, origin xyz=0 0 0 rpy=${-pi/2} 0 ${-pi/2}
- added joint zedm_mount_joint: type fixed, parent body_link, child zedm_camera_link, origin xyz=${body_length/2 - 0.0475} 0 ${0.02 - 0.0265/2} rpy=0 0 0

File: src/cobraflex/urdf/my_robot_mesh.urdf (robot description, URDF)
Before this commit: robot cobraflex_robot, 8 links, 7 joints
Links:
- added link camera_link_lane; collision cylinder length=0.002 radius=0.005; visual cylinder length=0.002 radius=0.005
- added link camera_link_optical_lane
Joints:
- added joint camera_joint_lane: type fixed, parent body_link, child camera_link_lane, origin xyz=${body_length/2 + 0.01} 0 -0.03 rpy=0 0.30 0
- added joint camera_optical_joint_lane: type fixed, parent camera_link_lane, child camera_link_optical_lane, origin xyz=0 0 0 rpy=${-pi/2} 0 ${-pi/2}
- joint body_joint: origin xyz=0 0 ${body_height/2 + chassis_height/2} -> xyz=0 0 ${body_height/2 + chassis_height/2 - 0.01}
- joint camera_joint: origin xyz=${body_length/2 - 0.04} 0 0.02 rpy=0 0 0 -> xyz=${body_length/2 - 0.0475} 0 0.02 rpy=0 0 0
- joint imu_joint: origin xyz=${body_length/2 - 0.04} 0 0.02 rpy=0 0 0 -> xyz=${body_length/2 - 0.0475} 0 0.02 rpy=0 0 0

File: src/cobraflex/urdf/zed_descr.urdf.xacro (robot description, xacro)
@@ -1,18 +1,3 @@
 <?xml version="1.0"?>
-<!--
-// Copyright 2025 Stereolabs
-//
-// Licensed under the Apache License, Version 2.0 (the "License");
-// you may not use this file except in compliance with the License.
-// You may obtain a copy of the License at
-//
-//      http://www.apache.org/licenses/LICENSE-2.0
-//
-// Unless required by applicable law or agreed to in writing, software
-// distributed under the License is distributed on an "AS IS" BASIS,
-// WITHOUT WARRANTIES OR CONDITIONS OF ANY KIND, either express or implied.
-// See the License for the specific language governing permissions and
-// limitations under the License.
--->
 <robot name="stereolabs_camera" xmlns:xacro="http://ros.org/wiki/xacro">
   <xacro:arg name="camera_name"   default="zed" />
@@ -25,5 +10,9 @@
   <xacro:arg name="gnss_z" default="0.0" />
   <xacro:include filename="$(find cobraflex)/urdf/zed_macro.urdf.xacro" />
-  <xacro:zed_camera name="$(arg camera_name)" model="$(arg camera_model)" custom_baseline="$(arg custom_baseline)" enable_gnss="$(arg enable_gnss)">
+  <!-- This wrapper is included ONLY by my_robot_basic.urdf, the RViz/hardware
+       description. mat_override lifts the zedm shell off rgba 0,0,0, which
+       RViz shades to an unlit void at the very front of the robot. The Gazebo
+       URDFs include zed_macro directly and so keep the stock colour. -->
+  <xacro:zed_camera name="$(arg camera_name)" model="$(arg camera_model)" custom_baseline="$(arg custom_baseline)" enable_gnss="$(arg enable_gnss)" mat_override="0.22 0.23 0.27 1.0">
 	    <origin xyz="$(arg gnss_x) $(arg gnss_y) $(arg gnss_z)" rpy="0 0 0"/>
   </xacro:zed_camera>

File: src/cobraflex/urdf/zed_macro.urdf.xacro (robot description, xacro)
@@ -23,5 +23,12 @@
       - enable_gnss: if true enable the URDF link
   -->
-  <xacro:macro name="zed_camera" params="name=zed model=zed enable_gnss=false custom_baseline=0 *gnss_origin">
+  <!-- mat_override: optional rgba replacing the per-model shell colour. The
+       default sentinel 'none' keeps every existing caller byte-identical -
+       my_robot_gazebo.urdf and my_robot_gazebo_mesh.urdf must NOT change,
+       because their cameras render this mesh and they are the models behind
+       the recorded campaign evidence. Only zed_descr.urdf.xacro (RViz /
+       hardware description) passes it, to lift the zedm shell off rgba 0,0,0,
+       which RViz shades to an unlit void. -->
+  <xacro:macro name="zed_camera" params="name=zed model=zed enable_gnss=false custom_baseline=0 mat_override=none *gnss_origin">
     <xacro:if value="${model == 'zed'}">
       <xacro:property name="baseline" value="0.12" />
@@ -153,4 +160,7 @@
       <xacro:property name="mono" value="true" />
       <xacro:property name="mat" value="0.25 0.25 0.25 1.0" />
+    </xacro:if>
+    <xacro:if value="${mat_override != 'none'}">
+      <xacro:property name="mat" value="${mat_override}" />
     </xacro:if>
     <!-- Camera mounting point (the threaded screw hole in the bottom) -->
@@ -205,5 +215,5 @@
         <parent link="${name}_camera_center"/>
         <child link="${name}_left_camera_frame"/>
-        <origin xyz="${optical_offset_x} ${baseline/2} 0" rpy="0 0 0" />
+        <origin xyz="${optical_offset_x + 0.02} ${baseline/2 - 0.007} 0" rpy="0 0 0" />
       </joint>
       <link name="${name}_left_camera_frame_optical"/>
@@ -236,5 +246,5 @@
         <parent link="${name}_camera_center"/>
         <child link="${name}_right_camera_frame"/>
-        <origin xyz="${optical_offset_x} -${baseline/2} 0" rpy="0 0 0" />
+        <origin xyz="${optical_offset_x + 0.02} -${baseline/2 + 0.007} 0" rpy="0 0 0" />
       </joint>
       <link name="${name}_right_camera_frame_optical"/>

Commit message: Repo Update

File: src/cobraflex/urdf/my_robot_basic.urdf (robot description, URDF)
Before this commit: robot cobraflex_robot, 23 links, 23 joints
Links:
- link body_link: mass None -> ${body_mass}

File: src/cobraflex/urdf/my_robot_gazebo.urdf (robot description, URDF)
Before this commit: robot cobraflex_robot, 7 links, 7 joints
Links:
- link body_link: mass None -> ${body_mass}

File: src/cobraflex/urdf/my_robot_gazebo_mesh.urdf (robot description, URDF)
Before this commit: robot cobraflex_robot, 7 links, 7 joints
Links:
- link body_link: mass None -> ${body_mass}

File: src/cobraflex/urdf/my_robot_mesh.urdf (robot description, URDF)
Before this commit: robot cobraflex_robot, 10 links, 9 joints
Links:
- link body_link: mass None -> ${body_mass}

Commit message: Cobraflex V4 update

File: src/cobraflex/urdf/my_robot_basic.urdf (robot description, URDF)
Before this commit: robot cobraflex_robot, 9 links, 9 joints
Links:
- link body_link: geometry collision box size=0.102 0.1299 0.057; collision box size=0.18 0.0995 0.0255

File: src/cobraflex/urdf/my_robot_gazebo.urdf (robot description, URDF)
Before this commit: robot cobraflex_robot, 7 links, 7 joints
Links:
- link body_link: geometry collision box size=0.102 0.1299 0.057; collision box size=0.18 0.0995 0.0255
